File: Yet-another-3d-printer-electronics/_saved_Power_section.sch (KiCad schematic (older format))
At the start: 26 parts, among them J2 CONN_01X02, J3 TEST_3.3V, J4 TEST_5V, J5 TEST_12V, U7 AP1501, U8 AP1501, U9 AP1501

Commit message: ADD DG300, EBBA-02 and fix DG638 connectors
Signed-off-by: Mateusz Krawczuk <mat.krawczuk@gmail.com>
Parts:
- J2: value CONN_01X02 -> DG638
Changed lines of the file:
@@
 P 9425 1700
 F 0 "J2" H 9425 1850 50  0000 C CNN
-F 1 "CONN_01X02" V 9525 1700 50  0000 C CNN
+F 1 "DG638" V 9525 1700 50  0000 C CNN
 F 2 "" H 9425 1700 50  0001 C CNN
 F 3 "" H 9425 1700 50  0001 C CNN
