File: Yet-another-3d-printer-electronics/Endstops.sch (KiCad schematic (older format))
At the start: 11 parts

Commit message: Add additional stepstick, hotend fan and heater and temperature sensor
Extruder stepsticks have independ enables pins. Vcc was replace by valid
power source.

Signed-off-by: Mateusz Krawczuk <mat.krawczuk@gmail.com>
Parts:
- gave numbers to parts that had none: 11
Changed lines of the file:
@@
 $Descr A4 11693 8268
 encoding utf-8
-Sheet 6 6
+Sheet 5 6
 Title ""
 Date ""
@@
 $EndDescr
 $Comp
-L CONN_01X03 P?
+L CONN_01X03 P17
 U 1 1 58FE0F8F
 P 1525 2325
-F 0 "P?" H 1525 2525 50  0000 C CNN
+F 0 "P17" H 1525 2525 50  0000 C CNN
 F 1 "X-ENDSTOP" V 1625 2325 50  0000 C CNN
 F 2 "Connectors_JST:JST_XH_B03B-XH-A_03x2.50mm_Straight" H 1525 2325 50  0001 C CNN
@@
 $EndComp
 $Comp
-L CONN_01X03 P?
+L CONN_01X03 P5
 U 1 1 58FE0F96
 P 1500 3050
-F 0 "P?" H 1500 3250 50  0000 C CNN
+F 0 "P5" H 1500 3250 50  0000 C CNN
 F 1 "Y-ENDSTOP" V 1600 3050 50  0000 C CNN
 F 2 "Connectors_JST:JST_XH_B03B-XH-A_03x2.50mm_Straight" H 1500 3050 50  0001 C CNN
@@
 	1725 2225 2250 2225
 $Comp
-L +5V #PWR?
+L +5V #PWR0101
 U 1 1 58FE125F
 P 2250 1850
-F 0 "#PWR?" H 2250 1700 50  0001 C CNN
+F 0 "#PWR0101" H 2250 1700 50  0001 C CNN
 F 1 "+5V" H 2250 1990 50  0000 C CNN
 F 2 "" H 2250 1850 50  0001 C CNN
@@
 Connection ~ 2250 2225
 $Comp
-L GND #PWR?
+L GND #PWR0102
 U 1 1 58FE131D
 P 1950 4375
-F 0 "#PWR?" H 1950 4125 50  0001 C CNN
+F 0 "#PWR0102" H 1950 4125 50  0001 C CNN
 F 1 "GND" H 1950 4225 50  0000 C CNN
 F 2 "" H 1950 4375 50  0000 C CNN
@@
 Connection ~ 1950 3050
 $Comp
-L CONN_01X03 P?
+L CONN_01X03 P6
 U 1 1 58FE139B
 P 1500 3800
-F 0 "P?" H 1500 4000 50  0000 C CNN
+F 0 "P6" H 1500 4000 50  0000 C CNN
 F 1 "Z-ENDSTOP" V 1600 3800 50  0000 C CNN
 F 2 "Connectors_JST:JST_XH_B03B-XH-A_03x2.50mm_Straight" H 1500 3800 50  0001 C CNN
@@
 	1725 2425 2375 2425
 $Comp
-L R R?
+L R R32
 U 1 1 58FE15AF
 P 2525 2425
-F 0 "R?" V 2605 2425 50  0000 C CNN
+F 0 "R32" V 2605 2425 50  0000 C CNN
 F 1 "R" V 2525 2425 50  0000 C CNN
 F 2 "" V 2455 2425 50  0001 C CNN
@@
 $EndComp
 $Comp
-L R R?
+L R R33
 U 1 1 58FE1633
 P 2525 3150
-F 0 "R?" V 2605 3150 50  0000 C CNN
+F 0 "R33" V 2605 3150 50  0000 C CNN
 F 1 "R" V 2525 3150 50  0000 C CNN
 F 2 "" V 2455 3150 50  0001 C CNN
@@
 $EndComp
 $Comp
-L R R?
+L R R34
 U 1 1 58FE168B
 P 2525 3900
-F 0 "R?" V 2605 3900 50  0000 C CNN
+F 0 "R34" V 2605 3900 50  0000 C CNN
 F 1 "R" V 2525 3900 50  0000 C CNN
 F 2 "" V 2455 3900 50  0001 C CNN
@@
 Connection ~ 2750 2425
 $Comp
-L C C?
+L C C25
 U 1 1 58FE1A07
 P 2750 2625
-F 0 "C?" H 2775 2725 50  0000 L CNN
+F 0 "C25" H 2775 2725 50  0000 L CNN
 F 1 "C" H 2775 2525 50  0000 L CNN
 F 2 "" H 2788 2475 50  0001 C CNN
@@
 	2750 2775 2750 2825
 $Comp
-L C C?
+L C C26
 U 1 1 58FE1A8F
 P 2750 3350
-F 0 "C?" H 2775 3450 50  0000 L CNN
+F 0 "C26" H 2775 3450 50  0000 L CNN
 F 1 "C" H 2775 3250 50  0000 L CNN
 F 2 "" H 2788 3200 50  0001 C CNN
@@
 Connection ~ 2750 3150
 $Comp
-L C C?
+L C C27
 U 1 1 58FE1B15
 P 2750 4100
-F 0 "C?" H 2775 4200 50  0000 L CNN
+F 0 "C27" H 2775 4200 50  0000 L CNN
 F 1 "C" H 2775 4000 50  0000 L CNN
 F 2 "" H 2788 3950 50  0001 C CNN
@@
 Connection ~ 2750 3900
 $Comp
-L GND #PWR?
+L GND #PWR0103
 U 1 1 58FE1C0C
 P 2750 2825
-F 0 "#PWR?" H 2750 2575 50  0001 C CNN
+F 0 "#PWR0103" H 2750 2575 50  0001 C CNN
 F 1 "GND" H 2750 2675 50  0000 C CNN
 F 2 "" H 2750 2825 50  0001 C CNN
@@
 $EndComp
 $Comp
-L GND #PWR?
+L GND #PWR0104
 U 1 1 58FE1C39
 P 2750 3550
-F 0 "#PWR?" H 2750 3300 50  0001 C CNN
+F 0 "#PWR0104" H 2750 3300 50  0001 C CNN
 F 1 "GND" H 2750 3400 50  0000 C CNN
 F 2 "" H 2750 3550 50  0001 C CNN
@@
 $EndComp
 $Comp
-L GND #PWR?
+L GND #PWR0105
 U 1 1 58FE1C5F
 P 2750 4300
-F 0 "#PWR?" H 2750 4050 50  0001 C CNN
+F 0 "#PWR0105" H 2750 4050 50  0001 C CNN
 F 1 "GND" H 2750 4150 50  0000 C CNN
 F 2 "" H 2750 4300 50  0001 C CNN
@@
 Connection ~ 2250 3700
 $Comp
-L C C?
+L C C23
 U 1 1 58FE1D8F
 P 2100 4050
-F 0 "C?" H 2125 4150 50  0000 L CNN
+F 0 "C23" H 2125 4150 50  0000 L CNN
 F 1 "C" H 2125 3950 50  0000 L CNN
 F 2 "" H 2138 3900 50  0001 C CNN
@@
 Connection ~ 2250 4050
 $Comp
-L C C?
+L C C24
 U 1 1 58FE1E35
 P 2100 4250
-F 0 "C?" H 2125 4350 50  0000 L CNN
+F 0 "C24" H 2125 4350 50  0000 L CNN
 F 1 "C" H 2125 4150 50  0000 L CNN
 F 2 "" H 2138 4100 50  0001 C CNN

Commit message: Add fuses to powersupply connector and heatbed.
TVS diode used to protect pins from short circuit. Correct connectors
names.

Signed-off-by: Mateusz Krawczuk <mat.krawczuk@gmail.com>
Parts:
- added D? (x3): D_TVS, symbol D_TVS
Connections:
- net ENDSTOP-X: now also D?.2 (A2); no longer C25.1, R32.1
- net ENDSTOP-Y: now also D?.2 (A2); no longer C26.1, R33.1
- net ENDSTOP-Z: now also D?.2 (A2); no longer C27.1, R34.1
- new net: C25.1, D?.1 (A1), R32.1
- new net: C26.1, D?.1 (A1), R33.1
- new net: C27.1, D?.1 (A1), R34.1
Changed lines of the file:
@@
 	2375 3900 1700 3900
 Wire Wire Line
-	2675 2425 2850 2425
+	2675 2425 3000 2425
 Wire Wire Line
-	2850 3150 2675 3150
+	2675 3150 3000 3150
 Wire Wire Line
-	2850 3900 2675 3900
+	2675 3900 3000 3900
 Wire Wire Line
 	2750 2425 2750 2475
@@
 Connection ~ 1950 4050
 Connection ~ 1950 4250
-Text HLabel 2850 2425 2    60   UnSpc ~ 0
+Text HLabel 3400 2425 2    60   UnSpc ~ 0
 ENDSTOP-X
-Text HLabel 2850 3150 2    60   UnSpc ~ 0
+Text HLabel 3425 3150 2    60   UnSpc ~ 0
 ENDSTOP-Y
-Text HLabel 2850 3900 2    60   UnSpc ~ 0
+Text HLabel 3450 3900 2    60   UnSpc ~ 0
 ENDSTOP-Z
+Wire Wire Line
+	3400 2425 3300 2425
+$Comp
+L D_TVS D?
+U 1 1 590459CA
+P 3150 2425
+F 0 "D?" H 3150 2525 50  0000 C CNN
+F 1 "D_TVS" H 3150 2325 50  0000 C CNN
+F 2 "" H 3150 2425 50  0001 C CNN
+F 3 "" H 3150 2425 50  0001 C CNN
+	1    3150 2425
+	1    0    0    -1
+$EndComp
+$Comp
+L D_TVS D?
+U 1 1 59045A23
+P 3150 3150
+F 0 "D?" H 3150 3250 50  0000 C CNN
+F 1 "D_TVS" H 3150 3050 50  0000 C CNN
+F 2 "" H 3150 3150 50  0001 C CNN
+F 3 "" H 3150 3150 50  0001 C CNN
+	1    3150 3150
+	1    0    0    -1
+$EndComp
+$Comp
+L D_TVS D?
+U 1 1 59045AB3
+P 3150 3900
+F 0 "D?" H 3150 4000 50  0000 C CNN
+F 1 "D_TVS" H 3150 3800 50  0000 C CNN
+F 2 "" H 3150 3900 50  0001 C CNN
+F 3 "" H 3150 3900 50  0001 C CNN
+	1    3150 3900
+	1    0    0    -1
+$EndComp
+Wire Wire Line
+	3450 3900 3300 3900
+Wire Wire Line
+	3425 3150 3300 3150
 $EndSCHEMATC

Commit message: Add programming jumper
Signed-off-by: Mateusz Krawczuk <mat.krawczuk@gmail.com>
Parts:
- gave numbers to parts that had none: 3
Changed lines of the file:
@@
 	1725 2225 2250 2225
 $Comp
-L +5V #PWR0101
+L +5V #PWR98
 U 1 1 58FE125F
 P 2250 1850
-F 0 "#PWR0101" H 2250 1700 50  0001 C CNN
+F 0 "#PWR98" H 2250 1700 50  0001 C CNN
 F 1 "+5V" H 2250 1990 50  0000 C CNN
 F 2 "" H 2250 1850 50  0001 C CNN
@@
 Connection ~ 2250 2225
 $Comp
-L GND #PWR0102
+L GND #PWR97
 U 1 1 58FE131D
 P 1950 4375
-F 0 "#PWR0102" H 1950 4125 50  0001 C CNN
+F 0 "#PWR97" H 1950 4125 50  0001 C CNN
 F 1 "GND" H 1950 4225 50  0000 C CNN
 F 2 "" H 1950 4375 50  0000 C CNN
@@
 Connection ~ 2750 3900
 $Comp
-L GND #PWR0103
+L GND #PWR99
 U 1 1 58FE1C0C
 P 2750 2825
-F 0 "#PWR0103" H 2750 2575 50  0001 C CNN
+F 0 "#PWR99" H 2750 2575 50  0001 C CNN
 F 1 "GND" H 2750 2675 50  0000 C CNN
 F 2 "" H 2750 2825 50  0001 C CNN
@@
 $EndComp
 $Comp
-L GND #PWR0104
+L GND #PWR100
 U 1 1 58FE1C39
 P 2750 3550
-F 0 "#PWR0104" H 2750 3300 50  0001 C CNN
+F 0 "#PWR100" H 2750 3300 50  0001 C CNN
 F 1 "GND" H 2750 3400 50  0000 C CNN
 F 2 "" H 2750 3550 50  0001 C CNN
@@
 $EndComp
 $Comp
-L GND #PWR0105
+L GND #PWR101
 U 1 1 58FE1C5F
 P 2750 4300
-F 0 "#PWR0105" H 2750 4050 50  0001 C CNN
+F 0 "#PWR101" H 2750 4050 50  0001 C CNN
 F 1 "GND" H 2750 4150 50  0000 C CNN
 F 2 "" H 2750 4300 50  0001 C CNN
@@
 	3400 2425 3300 2425
 $Comp
-L D_TVS D?
+L D_TVS D69
 U 1 1 590459CA
 P 3150 2425
-F 0 "D?" H 3150 2525 50  0000 C CNN
+F 0 "D69" H 3150 2525 50  0000 C CNN
 F 1 "D_TVS" H 3150 2325 50  0000 C CNN
 F 2 "" H 3150 2425 50  0001 C CNN
@@
 $EndComp
 $Comp
-L D_TVS D?
+L D_TVS D70
 U 1 1 59045A23
 P 3150 3150
-F 0 "D?" H 3150 3250 50  0000 C CNN
+F 0 "D70" H 3150 3250 50  0000 C CNN
 F 1 "D_TVS" H 3150 3050 50  0000 C CNN
 F 2 "" H 3150 3150 50  0001 C CNN
@@
 $EndComp
 $Comp
-L D_TVS D?
+L D_TVS D71
 U 1 1 59045AB3
 P 3150 3900
-F 0 "D?" H 3150 4000 50  0000 C CNN
+F 0 "D71" H 3150 4000 50  0000 C CNN
 F 1 "D_TVS" H 3150 3800 50  0000 C CNN
 F 2 "" H 3150 3900 50  0001 C CNN

Commit message: Choose footprints for some components
Signed-off-by: Mateusz Krawczuk <mat.krawczuk@gmail.com>
Parts:
- C23, C25, C26, C27: value C -> 100nF; footprint (none) -> Capacitors_SMD:C_0603_HandSoldering
- C24: value C -> 1uF; footprint (none) -> Capacitors_SMD:C_0805_HandSoldering
- R32, R33, R34: value R -> 10K; footprint (none) -> Resistors_SMD:R_0603_HandSoldering
Changed lines of the file:
@@
 	1725 2225 2250 2225
 $Comp
-L +5V #PWR98
+L +5V #PWR0102
 U 1 1 58FE125F
 P 2250 1850
-F 0 "#PWR98" H 2250 1700 50  0001 C CNN
+F 0 "#PWR0102" H 2250 1700 50  0001 C CNN
 F 1 "+5V" H 2250 1990 50  0000 C CNN
 F 2 "" H 2250 1850 50  0001 C CNN
@@
 Connection ~ 2250 2225
 $Comp
-L GND #PWR97
+L GND #PWR0103
 U 1 1 58FE131D
 P 1950 4375
-F 0 "#PWR97" H 1950 4125 50  0001 C CNN
+F 0 "#PWR0103" H 1950 4125 50  0001 C CNN
 F 1 "GND" H 1950 4225 50  0000 C CNN
 F 2 "" H 1950 4375 50  0000 C CNN
@@
 P 2525 2425
 F 0 "R32" V 2605 2425 50  0000 C CNN
-F 1 "R" V 2525 2425 50  0000 C CNN
-F 2 "" V 2455 2425 50  0001 C CNN
+F 1 "10K" V 2525 2425 50  0000 C CNN
+F 2 "Resistors_SMD:R_0603_HandSoldering" V 2455 2425 50  0001 C CNN
 F 3 "" H 2525 2425 50  0001 C CNN
 	1    2525 2425
@@
 P 2525 3150
 F 0 "R33" V 2605 3150 50  0000 C CNN
-F 1 "R" V 2525 3150 50  0000 C CNN
-F 2 "" V 2455 3150 50  0001 C CNN
+F 1 "10K" V 2525 3150 50  0000 C CNN
+F 2 "Resistors_SMD:R_0603_HandSoldering" V 2455 3150 50  0001 C CNN
 F 3 "" H 2525 3150 50  0001 C CNN
 	1    2525 3150
@@
 P 2525 3900
 F 0 "R34" V 2605 3900 50  0000 C CNN
-F 1 "R" V 2525 3900 50  0000 C CNN
-F 2 "" V 2455 3900 50  0001 C CNN
+F 1 "10K" V 2525 3900 50  0000 C CNN
+F 2 "Resistors_SMD:R_0603_HandSoldering" V 2455 3900 50  0001 C CNN
 F 3 "" H 2525 3900 50  0001 C CNN
 	1    2525 3900
@@
 P 2750 2625
 F 0 "C25" H 2775 2725 50  0000 L CNN
-F 1 "C" H 2775 2525 50  0000 L CNN
-F 2 "" H 2788 2475 50  0001 C CNN
+F 1 "100nF" H 2775 2525 50  0000 L CNN
+F 2 "Capacitors_SMD:C_0603_HandSoldering" H 2788 2475 50  0001 C CNN
 F 3 "" H 2750 2625 50  0001 C CNN
 	1    2750 2625
@@
 P 2750 3350
 F 0 "C26" H 2775 3450 50  0000 L CNN
-F 1 "C" H 2775 3250 50  0000 L CNN
-F 2 "" H 2788 3200 50  0001 C CNN
+F 1 "100nF" H 2775 3250 50  0000 L CNN
+F 2 "Capacitors_SMD:C_0603_HandSoldering" H 2788 3200 50  0001 C CNN
 F 3 "" H 2750 3350 50  0001 C CNN
 	1    2750 3350
@@
 P 2750 4100
 F 0 "C27" H 2775 4200 50  0000 L CNN
-F 1 "C" H 2775 4000 50  0000 L CNN
-F 2 "" H 2788 3950 50  0001 C CNN
+F 1 "100nF" H 2775 4000 50  0000 L CNN
+F 2 "Capacitors_SMD:C_0603_HandSoldering" H 2788 3950 50  0001 C CNN
 F 3 "" H 2750 4100 50  0001 C CNN
 	1    2750 4100
@@
 Connection ~ 2750 3900
 $Comp
-L GND #PWR99
+L GND #PWR0104
 U 1 1 58FE1C0C
 P 2750 2825
-F 0 "#PWR99" H 2750 2575 50  0001 C CNN
+F 0 "#PWR0104" H 2750 2575 50  0001 C CNN
 F 1 "GND" H 2750 2675 50  0000 C CNN
 F 2 "" H 2750 2825 50  0001 C CNN
@@
 $EndComp
 $Comp
-L GND #PWR100
+L GND #PWR0105
 U 1 1 58FE1C39
 P 2750 3550
-F 0 "#PWR100" H 2750 3300 50  0001 C CNN
+F 0 "#PWR0105" H 2750 3300 50  0001 C CNN
 F 1 "GND" H 2750 3400 50  0000 C CNN
 F 2 "" H 2750 3550 50  0001 C CNN
@@
 $EndComp
 $Comp
-L GND #PWR101
+L GND #PWR0106
 U 1 1 58FE1C5F
 P 2750 4300
-F 0 "#PWR101" H 2750 4050 50  0001 C CNN
+F 0 "#PWR0106" H 2750 4050 50  0001 C CNN
 F 1 "GND" H 2750 4150 50  0000 C CNN
 F 2 "" H 2750 4300 50  0001 C CNN
@@
 P 2100 4050
 F 0 "C23" H 2125 4150 50  0000 L CNN
-F 1 "C" H 2125 3950 50  0000 L CNN
-F 2 "" H 2138 3900 50  0001 C CNN
+F 1 "100nF" V 2150 3650 50  0000 L CNN
+F 2 "Capacitors_SMD:C_0603_HandSoldering" H 2138 3900 50  0001 C CNN
 F 3 "" H 2100 4050 50  0001 C CNN
 	1    2100 4050
@@
 P 2100 4250
 F 0 "C24" H 2125 4350 50  0000 L CNN
-F 1 "C" H 2125 4150 50  0000 L CNN
-F 2 "" H 2138 4100 50  0001 C CNN
+F 1 "1uF" V 2150 3900 50  0000 L CNN
+F 2 "Capacitors_SMD:C_0805_HandSoldering" H 2138 4100 50  0001 C CNN
 F 3 "" H 2100 4250 50  0001 C CNN
 	1    2100 4250

Commit message: Choose footprints for TVS diode, heatbed, heaters, power socket and testpoints
Signed-off-by: Mateusz Krawczuk <mat.krawczuk@gmail.com>
Parts:
- D69, D70, D71: footprint (none) -> Diodes_SMD:D_SOD-523
Changed lines of the file:
@@
 F 0 "D69" H 3150 2525 50  0000 C CNN
 F 1 "D_TVS" H 3150 2325 50  0000 C CNN
-F 2 "" H 3150 2425 50  0001 C CNN
+F 2 "Diodes_SMD:D_SOD-523" H 3150 2425 50  0001 C CNN
 F 3 "" H 3150 2425 50  0001 C CNN
 	1    3150 2425
@@
 F 0 "D70" H 3150 3250 50  0000 C CNN
 F 1 "D_TVS" H 3150 3050 50  0000 C CNN
-F 2 "" H 3150 3150 50  0001 C CNN
+F 2 "Diodes_SMD:D_SOD-523" H 3150 3150 50  0001 C CNN
 F 3 "" H 3150 3150 50  0001 C CNN
 	1    3150 3150
@@
 F 0 "D71" H 3150 4000 50  0000 C CNN
 F 1 "D_TVS" H 3150 3800 50  0000 C CNN
-F 2 "" H 3150 3900 50  0001 C CNN
+F 2 "Diodes_SMD:D_SOD-523" H 3150 3900 50  0001 C CNN
 F 3 "" H 3150 3900 50  0001 C CNN
 	1    3150 3900
