File: Yet-another-3d-printer-electronics/Power_section.sch (KiCad schematic (older format))
At the start: 23 parts, among them J2 CONN_01X02, U7 AP1501, U8 AP1501, U9 AP1501

Commit message: Choose footprints for some components
Signed-off-by: Mateusz Krawczuk <mat.krawczuk@gmail.com>
Parts:
- C17, C18, C19: value CP -> 100uF; footprint (none) -> Capacitors_SMD:CP_Elec_6.3x5.3
- C20, C21, C22: value CP -> 4,7uf; footprint (none) -> Capacitors_SMD:CP_Elec_6.3x5.3
- D43, D44, D45: footprint (none) -> Yet-another-3d-printer-electronics:DO-214AC(SMA)
- R26, R27, R28, R29, R30, R31: footprint (none) -> Resistors_SMD:R_1206_HandSoldering
- U7, U8, U9: footprint (none) -> TO_SOT_Packages_SMD:TO-263-5_TabPin3
Changed lines of the file:
@@
 $EndDescr
 $Comp
-L +24V #PWR83
+L +24V #PWR083
 U 1 1 58B11BCF
 P 2150 1900
-F 0 "#PWR83" H 2150 1750 50  0001 C CNN
+F 0 "#PWR083" H 2150 1750 50  0001 C CNN
 F 1 "+24V" H 2150 2040 50  0000 C CNN
 F 2 "" H 2150 1900 50  0000 C CNN
@@
 F 0 "U8" H 3200 1900 60  0000 C CNN
 F 1 "AP1501" H 3200 1800 60  0000 C CNN
-F 2 "" H 3200 1900 60  0001 C CNN
+F 2 "TO_SOT_Packages_SMD:TO-263-5_TabPin3" H 3200 1900 60  0001 C CNN
 F 3 "" H 3200 1900 60  0001 C CNN
 	1    3200 1900
@@
 P 2350 2200
 F 0 "C18" H 2375 2300 50  0000 L CNN
-F 1 "CP" H 2375 2100 50  0000 L CNN
-F 2 "" H 2388 2050 50  0001 C CNN
+F 1 "100uF" H 2375 2100 50  0000 L CNN
+F 2 "Capacitors_SMD:CP_Elec_6.3x5.3" H 2388 2050 50  0001 C CNN
 F 3 "" H 2350 2200 50  0001 C CNN
 	1    2350 2200
@@
 F 0 "D44" H 4050 2300 50  0000 C CNN
 F 1 "D_Schottky" H 4050 2100 50  0000 C CNN
-F 2 "" H 4050 2200 50  0001 C CNN
+F 2 "Yet-another-3d-printer-electronics:DO-214AC(SMA)" H 4050 2200 50  0001 C CNN
 F 3 "" H 4050 2200 50  0001 C CNN
 	1    4050 2200
@@
 P 4700 2200
 F 0 "C21" H 4725 2300 50  0000 L CNN
-F 1 "CP" H 4725 2100 50  0000 L CNN
-F 2 "" H 4738 2050 50  0001 C CNN
+F 1 "4,7uf" H 4725 2100 50  0000 L CNN
+F 2 "Capacitors_SMD:CP_Elec_6.3x5.3" H 4738 2050 50  0001 C CNN
 F 3 "" H 4700 2200 50  0001 C CNN
 	1    4700 2200
@@
 Connection ~ 4700 1900
 $Comp
-L +3.3V #PWR92
+L +3.3V #PWR084
 U 1 1 58FD74DD
 P 5100 1900
-F 0 "#PWR92" H 5100 1750 50  0001 C CNN
+F 0 "#PWR084" H 5100 1750 50  0001 C CNN
 F 1 "+3.3V" H 5100 2040 50  0000 C CNN
 F 2 "" H 5100 1900 50  0001 C CNN
@@
 $EndComp
 $Comp
-L GND #PWR89
+L GND #PWR085
 U 1 1 58FD7722
 P 3550 2450
-F 0 "#PWR89" H 3550 2200 50  0001 C CNN
+F 0 "#PWR085" H 3550 2200 50  0001 C CNN
 F 1 "GND" H 3550 2300 50  0000 C CNN
 F 2 "" H 3550 2450 50  0001 C CNN
@@
 $EndComp
 $Comp
-L GND #PWR86
+L GND #PWR086
 U 1 1 58FD7743
 P 2350 1600
-F 0 "#PWR86" H 2350 1350 50  0001 C CNN
+F 0 "#PWR086" H 2350 1350 50  0001 C CNN
 F 1 "GND" H 2350 1450 50  0000 C CNN
 F 2 "" H 2350 1600 50  0001 C CNN
@@
 F 0 "R30" V 3980 1450 50  0000 C CNN
 F 1 "R" V 3900 1450 50  0000 C CNN
-F 2 "" V 3830 1450 50  0001 C CNN
+F 2 "Resistors_SMD:R_1206_HandSoldering" V 3830 1450 50  0001 C CNN
 F 3 "" H 3900 1450 50  0001 C CNN
 	1    3900 1450
@@
 F 0 "R27" V 2880 1450 50  0000 C CNN
 F 1 "R" V 2800 1450 50  0000 C CNN
-F 2 "" V 2730 1450 50  0001 C CNN
+F 2 "Resistors_SMD:R_1206_HandSoldering" V 2730 1450 50  0001 C CNN
 F 3 "" H 2800 1450 50  0001 C CNN
 	1    2800 1450
@@
 	4050 2350 4050 2450
 $Comp
-L +24V #PWR84
+L +24V #PWR087
 U 1 1 58FD7B9F
 P 2150 3750
-F 0 "#PWR84" H 2150 3600 50  0001 C CNN
+F 0 "#PWR087" H 2150 3600 50  0001 C CNN
 F 1 "+24V" H 2150 3890 50  0000 C CNN
 F 2 "" H 2150 3750 50  0000 C CNN
@@
 F 0 "U9" H 3200 3750 60  0000 C CNN
 F 1 "AP1501" H 3200 3650 60  0000 C CNN
-F 2 "" H 3200 3750 60  0001 C CNN
+F 2 "TO_SOT_Packages_SMD:TO-263-5_TabPin3" H 3200 3750 60  0001 C CNN
 F 3 "" H 3200 3750 60  0001 C CNN
 	1    3200 3750
@@
 P 2350 4050
 F 0 "C19" H 2375 4150 50  0000 L CNN
-F 1 "CP" H 2375 3950 50  0000 L CNN
-F 2 "" H 2388 3900 50  0001 C CNN
+F 1 "100uF" H 2375 3950 50  0000 L CNN
+F 2 "Capacitors_SMD:CP_Elec_6.3x5.3" H 2388 3900 50  0001 C CNN
 F 3 "" H 2350 4050 50  0001 C CNN
 	1    2350 4050
@@
 F 0 "D45" H 4050 4150 50  0000 C CNN
 F 1 "D_Schottky" H 4050 3950 50  0000 C CNN
-F 2 "" H 4050 4050 50  0001 C CNN
+F 2 "Yet-another-3d-printer-electronics:DO-214AC(SMA)" H 4050 4050 50  0001 C CNN
 F 3 "" H 4050 4050 50  0001 C CNN
 	1    4050 4050
@@
 P 4700 4050
 F 0 "C22" H 4725 4150 50  0000 L CNN
-F 1 "CP" H 4725 3950 50  0000 L CNN
-F 2 "" H 4738 3900 50  0001 C CNN
+F 1 "4,7uf" H 4725 3950 50  0000 L CNN
+F 2 "Capacitors_SMD:CP_Elec_6.3x5.3" H 4738 3900 50  0001 C CNN
 F 3 "" H 4700 4050 50  0001 C CNN
 	1    4700 4050
@@
 Connection ~ 4700 3750
 $Comp
-L GND #PWR90
+L GND #PWR088
 U 1 1 58FD7BD8
 P 3550 4300
-F 0 "#PWR90" H 3550 4050 50  0001 C CNN
+F 0 "#PWR088" H 3550 4050 50  0001 C CNN
 F 1 "GND" H 3550 4150 50  0000 C CNN
 F 2 "" H 3550 4300 50  0001 C CNN
@@
 $EndComp
 $Comp
-L GND #PWR87
+L GND #PWR089
 U 1 1 58FD7BDE
 P 2350 3450
-F 0 "#PWR87" H 2350 3200 50  0001 C CNN
+F 0 "#PWR089" H 2350 3200 50  0001 C CNN
 F 1 "GND" H 2350 3300 50  0000 C CNN
 F 2 "" H 2350 3450 50  0001 C CNN
@@
 F 0 "R31" V 3980 3300 50  0000 C CNN
 F 1 "R" V 3900 3300 50  0000 C CNN
-F 2 "" V 3830 3300 50  0001 C CNN
+F 2 "Resistors_SMD:R_1206_HandSoldering" V 3830 3300 50  0001 C CNN
 F 3 "" H 3900 3300 50  0001 C CNN
 	1    3900 3300
@@
 F 0 "R28" V 2880 3300 50  0000 C CNN
 F 1 "R" V 2800 3300 50  0000 C CNN
-F 2 "" V 2730 3300 50  0001 C CNN
+F 2 "Resistors_SMD:R_1206_HandSoldering" V 2730 3300 50  0001 C CNN
 F 3 "" H 2800 3300 50  0001 C CNN
 	1    2800 3300
@@
 	4050 4200 4050 4300
 $Comp
-L +24V #PWR82
+L +24V #PWR090
 U 1 1 58FD7F6A
 P 2100 5650
-F 0 "#PWR82" H 2100 5500 50  0001 C CNN
+F 0 "#PWR090" H 2100 5500 50  0001 C CNN
 F 1 "+24V" H 2100 5790 50  0000 C CNN
 F 2 "" H 2100 5650 50  0000 C CNN
@@
 F 0 "U7" H 3150 5650 60  0000 C CNN
 F 1 "AP1501" H 3150 5550 60  0000 C CNN
-F 2 "" H 3150 5650 60  0001 C CNN
+F 2 "TO_SOT_Packages_SMD:TO-263-5_TabPin3" H 3150 5650 60  0001 C CNN
 F 3 "" H 3150 5650 60  0001 C CNN
 	1    3150 5650
@@
 P 2300 5950
 F 0 "C17" H 2325 6050 50  0000 L CNN
-F 1 "CP" H 2325 5850 50  0000 L CNN
-F 2 "" H 2338 5800 50  0001 C CNN
+F 1 "100uF" H 2325 5850 50  0000 L CNN
+F 2 "Capacitors_SMD:CP_Elec_6.3x5.3" H 2338 5800 50  0001 C CNN
 F 3 "" H 2300 5950 50  0001 C CNN
 	1    2300 5950
@@
 F 0 "D43" H 4000 6050 50  0000 C CNN
 F 1 "D_Schottky" H 4000 5850 50  0000 C CNN
-F 2 "" H 4000 5950 50  0001 C CNN
+F 2 "Yet-another-3d-printer-electronics:DO-214AC(SMA)" H 4000 5950 50  0001 C CNN
 F 3 "" H 4000 5950 50  0001 C CNN
 	1    4000 5950
@@
 P 4650 5950
 F 0 "C20" H 4675 6050 50  0000 L CNN
-F 1 "CP" H 4675 5850 50  0000 L CNN
-F 2 "" H 4688 5800 50  0001 C CNN
+F 1 "4,7uf" H 4675 5850 50  0000 L CNN
+F 2 "Capacitors_SMD:CP_Elec_6.3x5.3" H 4688 5800 50  0001 C CNN
 F 3 "" H 4650 5950 50  0001 C CNN
 	1    4650 5950
@@
 Connection ~ 4650 5650
 $Comp
-L GND #PWR88
+L GND #PWR091
 U 1 1 58FD7FA3
 P 3500 6200
-F 0 "#PWR88" H 3500 5950 50  0001 C CNN
+F 0 "#PWR091" H 3500 5950 50  0001 C CNN
 F 1 "GND" H 3500 6050 50  0000 C CNN
 F 2 "" H 3500 6200 50  0001 C CNN
@@
 $EndComp
 $Comp
-L GND #PWR85
+L GND #PWR092
 U 1 1 58FD7FA9
 P 2300 5350
-F 0 "#PWR85" H 2300 5100 50  0001 C CNN
+F 0 "#PWR092" H 2300 5100 50  0001 C CNN
 F 1 "GND" H 2300 5200 50  0000 C CNN
 F 2 "" H 2300 5350 50  0001 C CNN
@@
 F 0 "R29" V 3930 5200 50  0000 C CNN
 F 1 "R" V 3850 5200 50  0000 C CNN
-F 2 "" V 3780 5200 50  0001 C CNN
+F 2 "Resistors_SMD:R_1206_HandSoldering" V 3780 5200 50  0001 C CNN
 F 3 "" H 3850 5200 50  0001 C CNN
 	1    3850 5200
@@
 F 0 "R26" V 2830 5200 50  0000 C CNN
 F 1 "R" V 2750 5200 50  0000 C CNN
-F 2 "" V 2680 5200 50  0001 C CNN
+F 2 "Resistors_SMD:R_1206_HandSoldering" V 2680 5200 50  0001 C CNN
 F 3 "" H 2750 5200 50  0001 C CNN
 	1    2750 5200
@@
 	4000 6100 4000 6200
 $Comp
-L +5V #PWR93
+L +5V #PWR093
 U 1 1 58FD8102
 P 5100 3750
-F 0 "#PWR93" H 5100 3600 50  0001 C CNN
+F 0 "#PWR093" H 5100 3600 50  0001 C CNN
 F 1 "+5V" H 5100 3890 50  0000 C CNN
 F 2 "" H 5100 3750 50  0001 C CNN
@@
 $EndComp
 $Comp
-L +12V #PWR91
+L +12V #PWR094
 U 1 1 58FD82BA
 P 5050 5650
-F 0 "#PWR91" H 5050 5500 50  0001 C CNN
+F 0 "#PWR094" H 5050 5500 50  0001 C CNN
 F 1 "+12V" H 5050 5790 50  0000 C CNN
 F 2 "" H 5050 5650 50  0001 C CNN
@@
 $EndComp
 $Comp
-L +24V #PWR94
+L +24V #PWR095
 U 1 1 58FF7D10
 P 8025 1650
-F 0 "#PWR94" H 8025 1500 50  0001 C CNN
+F 0 "#PWR095" H 8025 1500 50  0001 C CNN
 F 1 "+24V" H 8025 1790 50  0000 C CNN
 F 2 "" H 8025 1650 50  0001 C CNN
@@
 	8800 1650 9225 1650
 $Comp
-L PWR_FLAG #FLG5
+L PWR_FLAG #FLG096
 U 1 1 58FF7EEB
 P 9100 1575
-F 0 "#FLG5" H 9100 1650 50  0001 C CNN
+F 0 "#FLG096" H 9100 1650 50  0001 C CNN
 F 1 "PWR_FLAG" H 9100 1725 50  0000 C CNN
 F 2 "" H 9100 1575 50  0001 C CNN
@@
 Connection ~ 9100 1650
 $Comp
-L GND #PWR95
+L GND #PWR097
 U 1 1 58FF7FE9
 P 8025 1750
-F 0 "#PWR95" H 8025 1500 50  0001 C CNN
+F 0 "#PWR097" H 8025 1500 50  0001 C CNN
 F 1 "GND" H 8025 1600 50  0000 C CNN
 F 2 "" H 8025 1750 50  0001 C CNN
@@
 	8025 1750 9225 1750
 $Comp
-L GNDPWR #PWR96
+L GNDPWR #PWR098
 U 1 1 58FF8089
 P 9100 1825
-F 0 "#PWR96" H 9100 1625 50  0001 C CNN
+F 0 "#PWR098" H 9100 1625 50  0001 C CNN
 F 1 "GNDPWR" H 9100 1695 50  0000 C CNN
 F 2 "" H 9100 1775 50  0001 C CNN
@@
 Connection ~ 9100 1750
 $Comp
-L PWR_FLAG #FLG3
+L PWR_FLAG #FLG099
 U 1 1 59003F28
 P 5000 3750
-F 0 "#FLG3" H 5000 3825 50  0001 C CNN
+F 0 "#FLG099" H 5000 3825 50  0001 C CNN
 F 1 "PWR_FLAG" H 5000 3900 50  0000 C CNN
 F 2 "" H 5000 3750 50  0001 C CNN
@@
 $EndComp
 $Comp
-L PWR_FLAG #FLG2
+L PWR_FLAG #FLG0100
 U 1 1 59003F75
 P 5000 1900
-F 0 "#FLG2" H 5000 1975 50  0001 C CNN
+F 0 "#FLG0100" H 5000 1975 50  0001 C CNN
 F 1 "PWR_FLAG" H 5000 2050 50  0000 C CNN
 F 2 "" H 5000 1900 50  0001 C CNN
@@
 $EndComp
 $Comp
-L PWR_FLAG #FLG4
+L PWR_FLAG #FLG0101
 U 1 1 590042F0
 P 5000 5650
-F 0 "#FLG4" H 5000 5725 50  0001 C CNN
+F 0 "#FLG0101" H 5000 5725 50  0001 C CNN
 F 1 "PWR_FLAG" H 5000 5800 50  0000 C CNN
 F 2 "" H 5000 5650 50  0001 C CNN

Commit message: Add testpoints to Heaters and Fans
Signed-off-by: Mateusz Krawczuk <mat.krawczuk@gmail.com>
Parts:
- added J?: TEST_3.3V, symbol TEST_1P
- added J?: TEST_5V, symbol TEST_1P
- added J?: TEST_12V, symbol TEST_1P
Connections:
- net +12V: now also J?.1
- net +3V3: now also J?.1
- net +5V: now also J?.1
Changed lines of the file:
@@
 LIBS:ap1501
 LIBS:Yet-another-3d-printer-electronics-cache
-EELAYER 25 0
+EELAYER 26 0
 EELAYER END
 $Descr A4 11693 8268
@@
 Wire Wire Line
 	8600 1650 8025 1650
+$Comp
+L TEST_1P J?
+U 1 1 5985A10E
+P 5000 2200
+F 0 "J?" H 4942 2227 50  0000 R CNN
+F 1 "TEST_3.3V" H 4942 2318 50  0000 R CNN
+F 2 "" H 5200 2200 50  0001 C CNN
+F 3 "" H 5200 2200 50  0001 C CNN
+	1    5000 2200
+	-1   0    0    1
+$EndComp
+Wire Wire Line
+	5000 2200 5000 1900
+Wire Wire Line
+	5000 3750 5000 4050
+$Comp
+L TEST_1P J?
+U 1 1 5985A2E6
+P 5000 4050
+F 0 "J?" H 4942 4077 50  0000 R CNN
+F 1 "TEST_5V" H 4942 4168 50  0000 R CNN
+F 2 "" H 5200 4050 50  0001 C CNN
+F 3 "" H 5200 4050 50  0001 C CNN
+	1    5000 4050
+	-1   0    0    1
+$EndComp
+Wire Wire Line
+	5000 5650 5000 5950
+$Comp
+L TEST_1P J?
+U 1 1 5985A7B5
+P 5000 5950
+F 0 "J?" H 4942 5977 50  0000 R CNN
+F 1 "TEST_12V" H 4942 6068 50  0000 R CNN
+F 2 "" H 5200 5950 50  0001 C CNN
+F 3 "" H 5200 5950 50  0001 C CNN
+	1    5000 5950
+	-1   0    0    1
+$EndComp
 $EndSCHEMATC

Commit message: Choose footprints for TVS diode, heatbed, heaters, power socket and testpoints
Signed-off-by: Mateusz Krawczuk <mat.krawczuk@gmail.com>
Parts:
- J2: value CONN_01X02 -> DG638; footprint (none) -> Yet-another-3d-printer-electronics:DG638-9.52-02P-14-00AH
- J3, J4, J5: renamed from J?; footprint (none) -> Connect:PINTST
Changed lines of the file:
@@
 P 9425 1700
 F 0 "J2" H 9425 1850 50  0000 C CNN
-F 1 "CONN_01X02" V 9525 1700 50  0000 C CNN
-F 2 "" H 9425 1700 50  0001 C CNN
+F 1 "DG638" V 9525 1700 50  0000 C CNN
+F 2 "Yet-another-3d-printer-electronics:DG638-9.52-02P-14-00AH" H 9425 1700 50  0001 C CNN
 F 3 "" H 9425 1700 50  0001 C CNN
 	1    9425 1700
@@
 	8600 1650 8025 1650
 $Comp
-L TEST_1P J?
+L TEST_1P J3
 U 1 1 5985A10E
 P 5000 2200
-F 0 "J?" H 4942 2227 50  0000 R CNN
+F 0 "J3" H 4942 2227 50  0000 R CNN
 F 1 "TEST_3.3V" H 4942 2318 50  0000 R CNN
-F 2 "" H 5200 2200 50  0001 C CNN
+F 2 "Connect:PINTST" H 5200 2200 50  0001 C CNN
 F 3 "" H 5200 2200 50  0001 C CNN
 	1    5000 2200
@@
 	5000 3750 5000 4050
 $Comp
-L TEST_1P J?
+L TEST_1P J4
 U 1 1 5985A2E6
 P 5000 4050
-F 0 "J?" H 4942 4077 50  0000 R CNN
+F 0 "J4" H 4942 4077 50  0000 R CNN
 F 1 "TEST_5V" H 4942 4168 50  0000 R CNN
-F 2 "" H 5200 4050 50  0001 C CNN
+F 2 "Connect:PINTST" H 5200 4050 50  0001 C CNN
 F 3 "" H 5200 4050 50  0001 C CNN
 	1    5000 4050
@@
 	5000 5650 5000 5950
 $Comp
-L TEST_1P J?
+L TEST_1P J5
 U 1 1 5985A7B5
 P 5000 5950
-F 0 "J?" H 4942 5977 50  0000 R CNN
+F 0 "J5" H 4942 5977 50  0000 R CNN
 F 1 "TEST_12V" H 4942 6068 50  0000 R CNN
-F 2 "" H 5200 5950 50  0001 C CNN
+F 2 "Connect:PINTST" H 5200 5950 50  0001 C CNN
 F 3 "" H 5200 5950 50  0001 C CNN
 	1    5000 5950
