File: Yet-another-3d-printer-electronics/Yet-another-3d-printer-electronics.sch (KiCad schematic (older format))
At the start: 29 parts, among them CON1 SD_Card, J1 LCD_Connector, P19 END2_TEMP, P2 BEDTEMP, P3 END1_TEMP, SW1 Switch_DPST, U2 LPC1114FBD48/302, X1 CRYSTAL_SMD

Commit message: Choose footprints for some components
Signed-off-by: Mateusz Krawczuk <mat.krawczuk@gmail.com>
Parts:
- R1, R2, R35, R7: footprint Resistors_SMD:R_0805_HandSoldering -> Resistors_SMD:R_0603_HandSoldering
Changed lines of the file:
@@
 RESET
 $Comp
-L GND #PWR17
+L GND #PWR01
 U 1 1 588666E7
 P 5675 5225
-F 0 "#PWR17" H 5675 4975 50  0001 C CNN
+F 0 "#PWR01" H 5675 4975 50  0001 C CNN
 F 1 "GND" H 5675 5075 50  0000 C CNN
 F 2 "" H 5675 5225 50  0000 C CNN
@@
 $EndComp
 $Comp
-L GND #PWR15
+L GND #PWR02
 U 1 1 5883A250
 P 5100 2325
-F 0 "#PWR15" H 5100 2075 50  0001 C CNN
+F 0 "#PWR02" H 5100 2075 50  0001 C CNN
 F 1 "GND" H 5100 2175 50  0000 C CNN
 F 2 "" H 5100 2325 50  0000 C CNN
@@
 $EndComp
 $Comp
-L GND #PWR10
+L GND #PWR03
 U 1 1 58852DAD
 P 3350 5100
-F 0 "#PWR10" H 3350 4850 50  0001 C CNN
+F 0 "#PWR03" H 3350 4850 50  0001 C CNN
 F 1 "GND" H 3350 4950 50  0000 C CNN
 F 2 "" H 3350 5100 50  0000 C CNN
@@
 F 0 "R7" V 4230 2475 50  0000 C CNN
 F 1 "R" V 4150 2475 50  0000 C CNN
-F 2 "Resistors_SMD:R_0805_HandSoldering" V 4080 2475 50  0001 C CNN
+F 2 "Resistors_SMD:R_0603_HandSoldering" V 4080 2475 50  0001 C CNN
 F 3 "" H 4150 2475 50  0000 C CNN
 	1    4150 2475
@@
 $EndComp
 $Comp
-L GND #PWR9
+L GND #PWR04
 U 1 1 58868622
 P 3325 3075
-F 0 "#PWR9" H 3325 2825 50  0001 C CNN
+F 0 "#PWR04" H 3325 2825 50  0001 C CNN
 F 1 "GND" H 3325 2925 50  0000 C CNN
 F 2 "" H 3325 3075 50  0000 C CNN
@@
 NoConn ~ 3050 6475
 $Comp
-L GND #PWR8
+L GND #PWR05
 U 1 1 588EF0E4
 P 3100 6900
-F 0 "#PWR8" H 3100 6650 50  0001 C CNN
+F 0 "#PWR05" H 3100 6650 50  0001 C CNN
 F 1 "GND" H 3100 6750 50  0000 C CNN
 F 2 "" H 3100 6900 50  0000 C CNN
@@
 $EndComp
 $Comp
-L GND #PWR2
+L GND #PWR06
 U 1 1 5890B49A
 P 1200 6475
-F 0 "#PWR2" H 1200 6225 50  0001 C CNN
+F 0 "#PWR06" H 1200 6225 50  0001 C CNN
 F 1 "GND" V 1200 6275 50  0000 C CNN
 F 2 "" H 1200 6475 50  0000 C CNN
@@
 SD-SS
 $Comp
-L GND #PWR4
+L GND #PWR07
 U 1 1 5890D76C
 P 1200 6775
-F 0 "#PWR4" H 1200 6525 50  0001 C CNN
+F 0 "#PWR07" H 1200 6525 50  0001 C CNN
 F 1 "GND" V 1200 6575 50  0000 C CNN
 F 2 "" H 1200 6775 50  0000 C CNN
@@
 $EndSheet
 $Comp
-L +3.3V #PWR16
+L +3.3V #PWR08
 U 1 1 58FDAA0A
 P 5675 2025
-F 0 "#PWR16" H 5675 1875 50  0001 C CNN
+F 0 "#PWR08" H 5675 1875 50  0001 C CNN
 F 1 "+3.3V" H 5675 2165 50  0000 C CNN
 F 2 "" H 5675 2025 50  0001 C CNN
@@
 Connection ~ 5675 2025
 $Comp
-L +3.3V #PWR11
+L +3.3V #PWR09
 U 1 1 58FDADD2
 P 4150 2275
-F 0 "#PWR11" H 4150 2125 50  0001 C CNN
+F 0 "#PWR09" H 4150 2125 50  0001 C CNN
 F 1 "+3.3V" H 4150 2415 50  0000 C CNN
 F 2 "" H 4150 2275 50  0001 C CNN
@@
 	2850 4375 4475 4375
 $Comp
-L +5V #PWR12
+L +5V #PWR010
 U 1 1 58FE5EAC
 P 4525 6425
-F 0 "#PWR12" H 4525 6275 50  0001 C CNN
+F 0 "#PWR010" H 4525 6275 50  0001 C CNN
 F 1 "+5V" H 4525 6565 50  0000 C CNN
 F 2 "" H 4525 6425 50  0001 C CNN
@@
 $EndComp
 $Comp
-L GND #PWR19
+L GND #PWR011
 U 1 1 58FE5F48
 P 5900 6425
-F 0 "#PWR19" H 5900 6175 50  0001 C CNN
+F 0 "#PWR011" H 5900 6175 50  0001 C CNN
 F 1 "GND" H 5900 6275 50  0000 C CNN
 F 2 "" H 5900 6425 50  0001 C CNN
@@
 	4475 4175 3675 4175
 $Comp
-L +3.3V #PWR3
+L +3.3V #PWR012
 U 1 1 5900DC8E
 P 1200 6575
-F 0 "#PWR3" H 1200 6425 50  0001 C CNN
+F 0 "#PWR012" H 1200 6425 50  0001 C CNN
 F 1 "+3.3V" H 1200 6715 50  0000 C CNN
 F 2 "" H 1200 6575 50  0001 C CNN
@@
 $EndComp
 $Comp
-L +3.3V #PWR6
+L +3.3V #PWR013
 U 1 1 5900830A
 P 2850 750
-F 0 "#PWR6" H 2850 600 50  0001 C CNN
+F 0 "#PWR013" H 2850 600 50  0001 C CNN
 F 1 "+3.3V" H 2850 890 50  0000 C CNN
 F 2 "" H 2850 750 50  0001 C CNN
@@
 END1_TEMP
 $Comp
-L GND #PWR7
+L GND #PWR014
 U 1 1 588E3505
 P 3025 1525
-F 0 "#PWR7" H 3025 1275 50  0001 C CNN
+F 0 "#PWR014" H 3025 1275 50  0001 C CNN
 F 1 "GND" H 3025 1375 50  0000 C CNN
 F 2 "" H 3025 1525 50  0000 C CNN
@@
 F 0 "R2" V 2930 925 50  0000 C CNN
 F 1 "10K" V 2850 925 50  0000 C CNN
-F 2 "Resistors_SMD:R_0805_HandSoldering" V 2780 925 50  0001 C CNN
+F 2 "Resistors_SMD:R_0603_HandSoldering" V 2780 925 50  0001 C CNN
 F 3 "" H 2850 925 50  0000 C CNN
 	1    2850 925
@@
 $EndComp
 $Comp
-L +3.3V #PWR1
+L +3.3V #PWR015
 U 1 1 59052ED6
 P 1150 750
-F 0 "#PWR1" H 1150 600 50  0001 C CNN
+F 0 "#PWR015" H 1150 600 50  0001 C CNN
 F 1 "+3.3V" H 1150 890 50  0000 C CNN
 F 2 "" H 1150 750 50  0001 C CNN
@@
 Connection ~ 1150 1125
 $Comp
-L GND #PWR5
+L GND #PWR016
 U 1 1 59052EE3
 P 1325 1525
-F 0 "#PWR5" H 1325 1275 50  0001 C CNN
+F 0 "#PWR016" H 1325 1275 50  0001 C CNN
 F 1 "GND" H 1325 1375 50  0000 C CNN
 F 2 "" H 1325 1525 50  0000 C CNN
@@
 F 0 "R1" V 1230 925 50  0000 C CNN
 F 1 "10K" V 1150 925 50  0000 C CNN
-F 2 "Resistors_SMD:R_0805_HandSoldering" V 1080 925 50  0001 C CNN
+F 2 "Resistors_SMD:R_0603_HandSoldering" V 1080 925 50  0001 C CNN
 F 3 "" H 1150 925 50  0000 C CNN
 	1    1150 925
@@
 	1800 1225 1800 1525
 $Comp
-L +3.3V #PWR13
+L +3.3V #PWR017
 U 1 1 59054E63
 P 4550 750
-F 0 "#PWR13" H 4550 600 50  0001 C CNN
+F 0 "#PWR017" H 4550 600 50  0001 C CNN
 F 1 "+3.3V" H 4550 890 50  0000 C CNN
 F 2 "" H 4550 750 50  0001 C CNN
@@
 Connection ~ 4550 1125
 $Comp
-L GND #PWR14
+L GND #PWR018
 U 1 1 59054E70
 P 4725 1525
-F 0 "#PWR14" H 4725 1275 50  0001 C CNN
+F 0 "#PWR018" H 4725 1275 50  0001 C CNN
 F 1 "GND" H 4725 1375 50  0000 C CNN
 F 2 "" H 4725 1525 50  0000 C CNN
@@
 F 0 "R35" V 4630 925 50  0000 C CNN
 F 1 "10K" V 4550 925 50  0000 C CNN
-F 2 "Resistors_SMD:R_0805_HandSoldering" V 4480 925 50  0001 C CNN
+F 2 "Resistors_SMD:R_0603_HandSoldering" V 4480 925 50  0001 C CNN
 F 3 "" H 4550 925 50  0000 C CNN
 	1    4550 925
@@
 $EndComp
 $Comp
-L GND #PWR18
+L GND #PWR019
 U 1 1 5905FBE0
 P 5675 7525
-F 0 "#PWR18" H 5675 7275 50  0001 C CNN
+F 0 "#PWR019" H 5675 7275 50  0001 C CNN
 F 1 "GND" H 5675 7375 50  0000 C CNN
 F 2 "" H 5675 7525 50  0001 C CNN

Commit message: Choose footprints for TVS diode, heatbed, heaters, power socket and testpoints
Signed-off-by: Mateusz Krawczuk <mat.krawczuk@gmail.com>
Parts:
- D58, D59, D60, D61, D62, D63, D64, D65, D66, D67, D68: footprint (none) -> Diodes_SMD:D_SOD-523
- J1: footprint (none) -> Pin_Headers:Pin_Header_Straight_2x05_Pitch2.54mm
- JP6: footprint (none) -> Pin_Headers:Pin_Header_Straight_1x02_Pitch2.54mm
Changed lines of the file:
@@
 F 0 "J1" H 4850 6925 50  0000 C CNN
 F 1 "LCD_Connector" H 4900 6325 50  0000 C CNN
-F 2 "" H 4850 5425 50  0001 C CNN
+F 2 "Pin_Headers:Pin_Header_Straight_2x05_Pitch2.54mm" H 4850 5425 50  0001 C CNN
 F 3 "" H 4850 5425 50  0001 C CNN
 	1    4850 6625
@@
 F 0 "D65" H 5150 6575 50  0000 C CNN
 F 1 "D_TVS" H 5300 6425 50  0001 C CNN
-F 2 "" H 5300 6525 50  0001 C CNN
+F 2 "Diodes_SMD:D_SOD-523" H 5300 6525 50  0001 C CNN
 F 3 "" H 5300 6525 50  0001 C CNN
 	1    5300 6525
@@
 F 0 "D66" H 5150 6675 50  0000 C CNN
 F 1 "D_TVS" H 5300 6525 50  0001 C CNN
-F 2 "" H 5300 6625 50  0001 C CNN
+F 2 "Diodes_SMD:D_SOD-523" H 5300 6625 50  0001 C CNN
 F 3 "" H 5300 6625 50  0001 C CNN
 	1    5300 6625
@@
 F 0 "D67" H 5150 6775 50  0000 C CNN
 F 1 "D_TVS" H 5300 6625 50  0001 C CNN
-F 2 "" H 5300 6725 50  0001 C CNN
+F 2 "Diodes_SMD:D_SOD-523" H 5300 6725 50  0001 C CNN
 F 3 "" H 5300 6725 50  0001 C CNN
 	1    5300 6725
@@
 F 0 "D68" H 5150 6875 50  0000 C CNN
 F 1 "D_TVS" H 5100 6725 50  0001 C CNN
-F 2 "" H 5300 6825 50  0001 C CNN
+F 2 "Diodes_SMD:D_SOD-523" H 5300 6825 50  0001 C CNN
 F 3 "" H 5300 6825 50  0001 C CNN
 	1    5300 6825
@@
 F 0 "D60" H 4225 6575 50  0000 C CNN
 F 1 "D_TVS" H 4375 6425 50  0001 C CNN
-F 2 "" H 4375 6525 50  0001 C CNN
+F 2 "Diodes_SMD:D_SOD-523" H 4375 6525 50  0001 C CNN
 F 3 "" H 4375 6525 50  0001 C CNN
 	1    4375 6525
@@
 F 0 "D61" H 4225 6675 50  0000 C CNN
 F 1 "D_TVS" H 4375 6525 50  0001 C CNN
-F 2 "" H 4375 6625 50  0001 C CNN
+F 2 "Diodes_SMD:D_SOD-523" H 4375 6625 50  0001 C CNN
 F 3 "" H 4375 6625 50  0001 C CNN
 	1    4375 6625
@@
 F 0 "D62" H 4225 6775 50  0000 C CNN
 F 1 "D_TVS" H 4375 6625 50  0001 C CNN
-F 2 "" H 4375 6725 50  0001 C CNN
+F 2 "Diodes_SMD:D_SOD-523" H 4375 6725 50  0001 C CNN
 F 3 "" H 4375 6725 50  0001 C CNN
 	1    4375 6725
@@
 F 0 "D63" H 4225 6875 50  0000 C CNN
 F 1 "D_TVS" H 4175 6725 50  0001 C CNN
-F 2 "" H 4375 6825 50  0001 C CNN
+F 2 "Diodes_SMD:D_SOD-523" H 4375 6825 50  0001 C CNN
 F 3 "" H 4375 6825 50  0001 C CNN
 	1    4375 6825
@@
 F 0 "D59" H 3350 1225 50  0000 C CNN
 F 1 "D_TVS" H 3350 1025 50  0000 C CNN
-F 2 "" H 3350 1125 50  0001 C CNN
+F 2 "Diodes_SMD:D_SOD-523" H 3350 1125 50  0001 C CNN
 F 3 "" H 3350 1125 50  0001 C CNN
 	1    3350 1125
@@
 F 0 "D58" H 1650 1225 50  0000 C CNN
 F 1 "D_TVS" H 1650 1025 50  0000 C CNN
-F 2 "" H 1650 1125 50  0001 C CNN
+F 2 "Diodes_SMD:D_SOD-523" H 1650 1125 50  0001 C CNN
 F 3 "" H 1650 1125 50  0001 C CNN
 	1    1650 1125
@@
 F 0 "D64" H 5050 1225 50  0000 C CNN
 F 1 "D_TVS" H 5050 1025 50  0000 C CNN
-F 2 "" H 5050 1125 50  0001 C CNN
+F 2 "Diodes_SMD:D_SOD-523" H 5050 1125 50  0001 C CNN
 F 3 "" H 5050 1125 50  0001 C CNN
 	1    5050 1125
@@
 F 0 "JP6" H 5675 7325 50  0000 C CNN
 F 1 "Prog jmp" H 5675 7095 50  0000 C CNN
-F 2 "" H 5675 7175 50  0001 C CNN
+F 2 "Pin_Headers:Pin_Header_Straight_1x02_Pitch2.54mm" H 5675 7175 50  0001 C CNN
 F 3 "" H 5675 7175 50  0001 C CNN
 	1    5675 7175
